File: ambika-smr4x.sch (EAGLE design)
At the start: 96 parts, among them IC1 TL074, IC2 LM13700N, IC3 LM13700N, IC4 LM13700N, IC5 TL072, IC6 MCP4822, IC7 ATMega328p, IC8 4052N, Q1 2N3906, Q2 2N3906, Q3 2N3906, Q4 2N3906, Q5 20MHz, Q6 2N7000, Q7 2N7000

Commit message: Updated original designer etc info in schematics
Updated original designer etc info in schematics
Other:
- note added: "Modifications by Björn Somell (bjoeri@gmail.com)"
- note added: "Original designer: Émilie Gillet (emilie.o.gillet@gmail.com)"
- note removed: "Original designer: Olivier Gillet (ol.gillet@gmail.com)"
- note removed: "This design by Björn Somell (bjoeri@gmail.com)"
